Commit message: chore: rename robotq_85 to robotiq_2f

File: robotiq_description/urdf/robotiq_2f_gripper.urdf.xacro (robot description, xacro)
@@ -1,20 +1,20 @@
 <?xml version="1.0"?>
-<robot name="robotiq_85_gripper" xmlns:xacro="http://www.ros.org/wiki/xacro">
-  <xacro:include filename="$(find robotiq_description)/urdf/robotiq_85_gripper.transmission.xacro" />
-  <xacro:macro name="robotiq_85_gripper" params="prefix parent *origin">
-    <joint name="${prefix}robotiq_85_base_joint" type="fixed">
+<robot name="robotiq_2f_gripper" xmlns:xacro="http://www.ros.org/wiki/xacro">
+  <xacro:include filename="$(find robotiq_description)/urdf/robotiq_2f_gripper.transmission.xacro" />
+  <xacro:macro name="robotiq_2f_gripper" params="prefix parent *origin">
+    <joint name="${prefix}robotiq_2f_base_joint" type="fixed">
       <parent link="${parent}"/>
-      <child link="${prefix}robotiq_85_base_link"/>
+      <child link="${prefix}robotiq_2f_base_link"/>
       <xacro:insert_block name="origin"/>
     </joint>
-    <link name="${prefix}robotiq_85_base_link">
-      <visual>
-        <geometry>
-          <mesh filename="package://robotiq_description/meshes/visual/robotiq_85_base_link.dae"/>
-        </geometry>
-      </visual>
-      <collision>
-        <geometry>
-          <mesh filename="package://robotiq_description/meshes/collision/robotiq_85_base_link.stl"/>
+    <link name="${prefix}robotiq_2f_base_link">
+      <visual>
+        <geometry>
+          <mesh filename="package://robotiq_description/meshes/visual/robotiq_2f_base_link.dae"/>
+        </geometry>
+      </visual>
+      <collision>
+        <geometry>
+          <mesh filename="package://robotiq_description/meshes/collision/robotiq_2f_base_link.stl"/>
         </geometry>
       </collision>
@@ -27,28 +27,28 @@
       </inertial>
     </link>
-    <joint name="${prefix}robotiq_85_left_knuckle_joint" type="revolute">
-      <parent link="${prefix}robotiq_85_base_link"/>
-      <child link="${prefix}robotiq_85_left_knuckle_link"/>
+    <joint name="${prefix}robotiq_2f_left_knuckle_joint" type="revolute">
+      <parent link="${prefix}robotiq_2f_base_link"/>
+      <child link="${prefix}robotiq_2f_left_knuckle_link"/>
       <axis xyz="0 0 1"/>
       <origin rpy="${pi} 0.0 0.0" xyz="0.05490451627 0.03060114443 0.0"/>
       <limit lower="0.0" upper="0.80285" velocity="0.5" effort="1000"/>
     </joint>
-    <joint name="${prefix}robotiq_85_right_knuckle_joint" type="continuous">
-      <parent link="${prefix}robotiq_85_base_link"/>
-      <child link="${prefix}robotiq_85_right_knuckle_link"/>
+    <joint name="${prefix}robotiq_2f_right_knuckle_joint" type="continuous">
+      <parent link="${prefix}robotiq_2f_base_link"/>
+      <child link="${prefix}robotiq_2f_right_knuckle_link"/>
       <axis xyz="0 0 1"/>
       <origin rpy="0.0 0.0 0.0" xyz="0.05490451627 -0.03060114443 0.0"/>
       <limit lower="-3.14" upper="3.14" velocity="100.0" effort="1000"/>
-      <mimic joint="${prefix}robotiq_85_left_knuckle_joint"/>
-    </joint>
-    <link name="${prefix}robotiq_85_left_knuckle_link">
-      <visual>
-        <geometry>
-          <mesh filename="package://robotiq_description/meshes/visual/robotiq_85_knuckle_link.dae"/>
-        </geometry>
-      </visual>
-      <collision>
-        <geometry>
-          <mesh filename="package://robotiq_description/meshes/collision/robotiq_85_knuckle_link.stl"/>
+      <mimic joint="${prefix}robotiq_2f_left_knuckle_joint"/>
+    </joint>
+    <link name="${prefix}robotiq_2f_left_knuckle_link">
+      <visual>
+        <geometry>
+          <mesh filename="package://robotiq_description/meshes/visual/robotiq_2f_knuckle_link.dae"/>
+        </geometry>
+      </visual>
+      <collision>
+        <geometry>
+          <mesh filename="package://robotiq_description/meshes/collision/robotiq_2f_knuckle_link.stl"/>
         </geometry>
       </collision>
@@ -61,13 +61,13 @@
       </inertial>
     </link>
-    <link name="${prefix}robotiq_85_right_knuckle_link">
-      <visual>
-        <geometry>
-          <mesh filename="package://robotiq_description/meshes/visual/robotiq_85_knuckle_link.dae"/>
-        </geometry>
-      </visual>
-      <collision>
-        <geometry>
-          <mesh filename="package://robotiq_description/meshes/collision/robotiq_85_knuckle_link.stl"/>
+    <link name="${prefix}robotiq_2f_right_knuckle_link">
+      <visual>
+        <geometry>
+          <mesh filename="package://robotiq_description/meshes/visual/robotiq_2f_knuckle_link.dae"/>
+        </geometry>
+      </visual>
+      <collision>
+        <geometry>
+          <mesh filename="package://robotiq_description/meshes/collision/robotiq_2f_knuckle_link.stl"/>
         </geometry>
       </collision>
@@ -80,23 +80,23 @@
       </inertial>
     </link>
-    <joint name="${prefix}robotiq_85_left_finger_joint" type="fixed">
-      <parent link="${prefix}robotiq_85_left_knuckle_link"/>
-      <child link="${prefix}robotiq_85_left_finger_link"/>
+    <joint name="${prefix}robotiq_2f_left_finger_joint" type="fixed">
+      <parent link="${prefix}robotiq_2f_left_knuckle_link"/>
+      <child link="${prefix}robotiq_2f_left_finger_link"/>
       <origin xyz="-0.00408552455 -0.03148604435 0.0" rpy="0 0 0" />
     </joint>
-    <joint name="${prefix}robotiq_85_right_finger_joint" type="fixed">
-      <parent link="${prefix}robotiq_85_right_knuckle_link"/>
-      <child link="${prefix}robotiq_85_right_finger_link"/>
+    <joint name="${prefix}robotiq_2f_right_finger_joint" type="fixed">
+      <parent link="${prefix}robotiq_2f_right_knuckle_link"/>
+      <child link="${prefix}robotiq_2f_right_finger_link"/>
       <origin xyz="-0.00408552455 -0.03148604435 0.0" rpy="0 0 0" />
     </joint>
-    <link name="${prefix}robotiq_85_left_finger_link">
-      <visual>
-        <geometry>
-          <mesh filename="package://robotiq_description/meshes/visual/robotiq_85_finger_link.dae"/>
-        </geometry>
-      </visual>
-      <collision>
-        <geometry>
-          <mesh filename="package://robotiq_description/meshes/collision/robotiq_85_finger_link.stl"/>
+    <link name="${prefix}robotiq_2f_left_finger_link">
+      <visual>
+        <geometry>
+          <mesh filename="package://robotiq_description/meshes/visual/robotiq_2f_finger_link.dae"/>
+        </geometry>
+      </visual>
+      <collision>
+        <geometry>
+          <mesh filename="package://robotiq_description/meshes/collision/robotiq_2f_finger_link.stl"/>
         </geometry>
       </collision>
@@ -109,13 +109,13 @@
       </inertial>
     </link>
-    <link name="${prefix}robotiq_85_right_finger_link">
-      <visual>
-        <geometry>
-          <mesh filename="package://robotiq_description/meshes/visual/robotiq_85_finger_link.dae"/>
-        </geometry>
-      </visual>
-      <collision>
-        <geometry>
-          <mesh filename="package://robotiq_description/meshes/collision/robotiq_85_finger_link.stl"/>
+    <link name="${prefix}robotiq_2f_right_finger_link">
+      <visual>
+        <geometry>
+          <mesh filename="package://robotiq_description/meshes/visual/robotiq_2f_finger_link.dae"/>
+        </geometry>
+      </visual>
+      <collision>
+        <geometry>
+          <mesh filename="package://robotiq_description/meshes/collision/robotiq_2f_finger_link.stl"/>
         </geometry>
       </collision>
@@ -128,29 +128,29 @@
       </inertial>
     </link>
-    <joint name="${prefix}robotiq_85_left_inner_knuckle_joint" type="continuous">
-      <parent link="${prefix}robotiq_85_base_link"/>
-      <child link="${prefix}robotiq_85_left_inner_knuckle_link"/>
+    <joint name="${prefix}robotiq_2f_left_inner_knuckle_joint" type="continuous">
+      <parent link="${prefix}robotiq_2f_base_link"/>
+      <child link="${prefix}robotiq_2f_left_inner_knuckle_link"/>
       <axis xyz="0 0 1"/>
       <origin xyz="0.06142 0.0127 0" rpy="${pi} 0.0 0.0" />
       <limit lower="-3.14" upper="3.14" velocity="100.0" effort="0.1"/>
-      <mimic joint="${prefix}robotiq_85_left_knuckle_joint" offset="0"/>
-    </joint>
-    <joint name="${prefix}robotiq_85_right_inner_knuckle_joint" type="continuous">
-      <parent link="${prefix}robotiq_85_base_link"/>
-      <child link="${prefix}robotiq_85_right_inner_knuckle_link"/>
+      <mimic joint="${prefix}robotiq_2f_left_knuckle_joint" offset="0"/>
+    </joint>
+    <joint name="${prefix}robotiq_2f_right_inner_knuckle_joint" type="continuous">
+      <parent link="${prefix}robotiq_2f_base_link"/>
+      <child link="${prefix}robotiq_2f_right_inner_knuckle_link"/>
       <axis xyz="0 0 1"/>
       <origin xyz="0.06142 -0.0127 0" rpy="0 0 0"/>
       <limit lower="-3.14" upper="3.14" velocity="100.0" effort="0.1"/>
-      <mimic joint="${prefix}robotiq_85_left_knuckle_joint" offset="0"/>
-    </joint>
-    <link name="${prefix}robotiq_85_left_inner_knuckle_link">
-      <visual>
-        <geometry>
-          <mesh filename="package://robotiq_description/meshes/visual/robotiq_85_inner_knuckle_link.dae"/>
-        </geometry>
-      </visual>
-      <collision>
-        <geometry>
-          <mesh filename="package://robotiq_description/meshes/collision/robotiq_85_inner_knuckle_link.stl"/>
+      <mimic joint="${prefix}robotiq_2f_left_knuckle_joint" offset="0"/>
+    </joint>
+    <link name="${prefix}robotiq_2f_left_inner_knuckle_link">
+      <visual>
+        <geometry>
+          <mesh filename="package://robotiq_description/meshes/visual/robotiq_2f_inner_knuckle_link.dae"/>
+        </geometry>
+      </visual>
+      <collision>
+        <geometry>
+          <mesh filename="package://robotiq_description/meshes/collision/robotiq_2f_inner_knuckle_link.stl"/>
         </geometry>
       </collision>
@@ -163,13 +163,13 @@
       </inertial>
     </link>
-    <link name="${prefix}robotiq_85_right_inner_knuckle_link">
-      <visual>
-        <geometry>
-          <mesh filename="package://robotiq_description/meshes/visual/robotiq_85_inner_knuckle_link.dae"/>
-        </geometry>
-      </visual>
-      <collision>
-        <geometry>
-          <mesh filename="package://robotiq_description/meshes/collision/robotiq_85_inner_knuckle_link.stl"/>
+    <link name="${prefix}robotiq_2f_right_inner_knuckle_link">
+      <visual>
+        <geometry>
+          <mesh filename="package://robotiq_description/meshes/visual/robotiq_2f_inner_knuckle_link.dae"/>
+        </geometry>
+      </visual>
+      <collision>
+        <geometry>
+          <mesh filename="package://robotiq_description/meshes/collision/robotiq_2f_inner_knuckle_link.stl"/>
         </geometry>
       </collision>
@@ -182,29 +182,29 @@
       </inertial>
     </link>
-    <joint name="${prefix}robotiq_85_left_finger_tip_joint" type="continuous">
-      <parent link="${prefix}robotiq_85_left_inner_knuckle_link"/>
-      <child link="${prefix}robotiq_85_left_finger_tip_link"/>
+    <joint name="${prefix}robotiq_2f_left_finger_tip_joint" type="continuous">
+      <parent link="${prefix}robotiq_2f_left_inner_knuckle_link"/>
+      <child link="${prefix}robotiq_2f_left_finger_tip_link"/>
       <axis xyz="0 0 1"/>
       <origin xyz="0.04303959807 -0.03759940821 0.0" rpy="0.0 0.0 0.0"/>
       <limit lower="-3.14" upper="3.14" velocity="100.0" effort="0.1"/>
-      <mimic joint="${prefix}robotiq_85_left_knuckle_joint" multiplier="-1"/>
-    </joint>
-    <joint name="${prefix}robotiq_85_right_finger_tip_joint" type="continuous">
-      <parent link="${prefix}robotiq_85_right_inner_knuckle_link"/>
-      <child link="${prefix}robotiq_85_right_finger_tip_link"/>
+      <mimic joint="${prefix}robotiq_2f_left_knuckle_joint" multiplier="-1"/>
+    </joint>
+    <joint name="${prefix}robotiq_2f_right_finger_tip_joint" type="continuous">
+      <parent link="${prefix}robotiq_2f_right_inner_knuckle_link"/>
+      <child link="${prefix}robotiq_2f_right_finger_tip_link"/>
       <axis xyz="0 0 1"/>
       <origin rpy="0.0 0.0 0.0" xyz="0.04303959807 -0.03759940821  0.0"/>
       <limit lower="-3.14" upper="3.14" velocity="100.0" effort="0.1"/>
-      <mimic joint="${prefix}robotiq_85_left_knuckle_joint" multiplier="-1"/>
-    </joint>
-    <link name="${prefix}robotiq_85_left_finger_tip_link">
-      <visual>
-        <geometry>
-          <mesh filename="package://robotiq_description/meshes/visual/robotiq_85_finger_tip_link.dae"/>
-        </geometry>
-      </visual>
-      <collision>
-        <geometry>
-          <mesh filename="package://robotiq_description/meshes/collision/robotiq_85_finger_tip_link.stl"/>
+      <mimic joint="${prefix}robotiq_2f_left_knuckle_joint" multiplier="-1"/>
+    </joint>
+    <link name="${prefix}robotiq_2f_left_finger_tip_link">
+      <visual>
+        <geometry>
+          <mesh filename="package://robotiq_description/meshes/visual/robotiq_2f_finger_tip_link.dae"/>
+        </geometry>
+      </visual>
+      <collision>
+        <geometry>
+          <mesh filename="package://robotiq_description/meshes/collision/robotiq_2f_finger_tip_link.stl"/>
         </geometry>
       </collision>
@@ -217,13 +217,13 @@
       </inertial>
     </link>
-    <link name="${prefix}robotiq_85_right_finger_tip_link">
-      <visual>
-        <geometry>
-          <mesh filename="package://robotiq_description/meshes/visual/robotiq_85_finger_tip_link.dae"/>
-        </geometry>
-      </visual>
-      <collision>
-        <geometry>
-          <mesh filename="package://robotiq_description/meshes/collision/robotiq_85_finger_tip_link.stl"/>
+    <link name="${prefix}robotiq_2f_right_finger_tip_link">
+      <visual>
+        <geometry>
+          <mesh filename="package://robotiq_description/meshes/visual/robotiq_2f_finger_tip_link.dae"/>
+        </geometry>
+      </visual>
+      <collision>
+        <geometry>
+          <mesh filename="package://robotiq_description/meshes/collision/robotiq_2f_finger_tip_link.stl"/>
         </geometry>
       </collision>
@@ -237,5 +237,5 @@
     </link>
     <!-- Improve grasping physics -->
-    <gazebo reference="${prefix}robotiq_85_left_finger_tip_link">
+    <gazebo reference="${prefix}robotiq_2f_left_finger_tip_link">
       <kp>1000000.0</kp>
       <kd>1.0</kd>
@@ -244,5 +244,5 @@
       <minDepth>0.001</minDepth>
     </gazebo>
-    <gazebo reference="${prefix}robotiq_85_right_finger_tip_link">
+    <gazebo reference="${prefix}robotiq_2f_right_finger_tip_link">
       <kp>1000000.0</kp>
       <kd>1.0</kd>
@@ -251,5 +251,5 @@
       <minDepth>0.001</minDepth>
     </gazebo>
-    <xacro:robotiq_85_gripper_transmission prefix="${prefix}" />
+    <xacro:robotiq_2f_gripper_transmission prefix="${prefix}" />
   </xacro:macro>
 </robot>

File: robotiq_description/urdf/robotiq_2f_gripper.xacro (robot description, xacro)
@@ -1,5 +1,5 @@
 <?xml version="1.0" ?>
-<robot name="robotiq_85_gripper" xmlns:xacro="http://www.ros.org/wiki/xacro">
-  <xacro:include filename="$(find robotiq_description)/urdf/robotiq_85_gripper.urdf.xacro" />
+<robot name="robotiq_2f_gripper" xmlns:xacro="http://www.ros.org/wiki/xacro">
+  <xacro:include filename="$(find robotiq_description)/urdf/robotiq_2f_gripper.urdf.xacro" />
   <gazebo>
     <plugin name="gazebo_ros_control" filename="libgazebo_ros_control.so">
@@ -34,6 +34,6 @@
     </inertial>
   </link>
-  <xacro:robotiq_85_gripper prefix="" parent="gripper_root_link" >
+  <xacro:robotiq_2f_gripper prefix="" parent="gripper_root_link" >
     <origin xyz="0.05 0 0.85" rpy="0 0 0"/>
-  </xacro:robotiq_85_gripper>
+  </xacro:robotiq_2f_gripper>
 </robot>

File: robotiq_description/urdf/robotiq_2f_gripper_sim_base.urdf.xacro (robot description, xacro)
@@ -1,5 +1,5 @@
 <?xml version="1.0"?>
-<robot name="robotiq_85_gripper_sim_base" xmlns:xacro="http://www.ros.org/wiki/xacro">
-  <xacro:macro name="robotiq_85_gripper_sim_base" params="prefix">
+<robot name="robotiq_2f_gripper_sim_base" xmlns:xacro="http://www.ros.org/wiki/xacro">
+  <xacro:macro name="robotiq_2f_gripper_sim_base" params="prefix">
     <link name="${prefix}gripper_root_link">
       <visual>
